File: pcb/vhf-am-tx/vhf-am-tx.kicad_sch (KiCad schematic)
At the start: 165 parts, among them J1 Conn_01x02_Pin, J10 AQM0802A-RN-GBW_Pin, J11 Jamper, J12 Jamper, J13 Jamper, J14 Conn_Coaxial, J2 Conn_01x02_Pin, J3 Conn_01x02_Pin, J4 SW_Power, J5 Conn_01x02_Pin, J6 Conn_01x04_Pin, J7 Conn_01x04_Pin, J8 NJW4190M, J9 SPU0414HR5H-SB Module, Q1 SSM3J334R, Q2 2SK4017, Q3 2SC4703, Q4 HTL7G06S006P, SW1 SW_Push, SW2 SW_Push, SW3 SW_Push, U1 XIAO-ESP32-C6, U2 NJM2125F, U3 Si5351a Module, U4 RT8250GSP, U5 BP5293-33, U6 NJM78L33SU3

Commit message: ドキュメント更新
Parts:
- C39: value 10p -> 3p; now fitted
- L7: value 56n -> 24n
Other:
- moved on the sheet: C37, L6
